Commit message: lab2

File: urdf/urdf_from_xacro.urdf (robot description, URDF)
Before this commit: robot navvis, 11 links, 10 joints
Links:
- removed link laser_horiz_joint
- removed link laser_vert_bottom_link
- removed link laser_vert_bottom_link_1
- removed link laser_vert_top_left_joint
- removed link laser_vert_top_right_joint
- removed link wheel_center_joint
- removed link wheel_left_joint
- removed link wheel_right_joint
- added link laser_vert_bottom, mass 1e-5; collision box size=0.1 0.1 0.1; visual mesh filename=package://gazebo_plugins/test/multi_robot_scenario/meshes/l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
- added link laser_vert_top_left, mass 1e-5; collision box size=0.1 0.1 0.1; visual mesh filename=package://gazebo_plugins/test/multi_robot_scenario/meshes/l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
- added link laser_vert_top_right, mass 1e-5; collision box size=0.1 0.1 0.1; visual mesh filename=package://gazebo_plugins/test/multi_robot_scenario/meshes/l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
- added link wheel_center; collision cylinder length=0.05 radius=0.15; visual cylinder length=0.05 radius=0.15
- added link wheel_left; collision cylinder length=0.05 radius=0.2; visual cylinder length=0.05 radius=0.2
- added link wheel_right; collision cylinder length=0.05 radius=0.2; visual cylinder length=0.05 radius=0.2
Joints:
- removed joint base_laser_horiz_joint
- removed joint base_laser_vert_bottom_link_1_joint
- joint base_laser_vert_bottom_joint: axis (none) -> 0 0 1; child laser_vert_bottom_link -> laser_vert_bottom; origin xyz=0.3158 -0.0021 0.5100 rpy=3.1355 -1.3045 0.0025 -> xyz=0.3157894464801903 -0.002068548615034871 0.5099999434059285 rpy=3.1354753 -1.3045001 0.0024658
- joint base_laser_vert_top_left_joint: axis (none) -> 0 0 1; child laser_vert_top_left_joint -> laser_vert_top_left
- joint base_laser_vert_top_right_joint: axis (none) -> 0 0 1; child laser_vert_top_right_joint -> laser_vert_top_right
- joint base_wheel_center_joint: axis (none) -> 0.0 0.0 1.0; child wheel_center_joint -> wheel_center; limit (none) -> effort=10.0 velocity=10.0; origin xyz=0.10 0.0 0.0 rpy=-1.5707 0.0 0.0 -> xyz=0.10 0.0 -0.05 rpy=-1.5707963267948966 0.0 0.0; type fixed -> continuous
- joint base_wheel_left_joint: axis 0 0 1 -> 0.0 0.0 1.0; child wheel_left_joint -> wheel_left; limit effort=1000000.0 velocity=1000000.0 -> effort=10.0 velocity=10.0; origin xyz=-0.10 0.4 0.0 rpy=-1.5707 0.0 0.0 -> xyz=-0.10 0.4 0.0 rpy=-1.5707963267948966 0.0 0.0
- joint base_wheel_right_joint: axis 0 0 1 -> 0.0 0.0 1.0; child wheel_right_joint -> wheel_right; limit effort=1000000.0 velocity=1000000.0 -> effort=10.0 velocity=10.0; origin xyz=-0.10 -0.4 0.0 rpy=-1.5707 0.0 0.0 -> xyz=-0.10 -0.4 0.0 rpy=-1.5707963267948966 0.0 0.0
